File: Power-Monitoring-Board/Power-Monitoring-Board.kicad_pcb (KiCad board)
At the start: 2 copper layers, 127 x 72 mm, 47 parts, among them IC1 XC6222D331MR-G, J1 Conn_01x02_Pin, J2 Conn_01x02_Pin, J3 Conn_01x01_Pin, J4 Conn_01x01_Pin, J5 Conn_01x01_Pin, J6 Conn_01x01_Pin, J7 Conn_01x02_Pin, J8 Conn_01x02_Pin, SW1 GF-123-0054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

Commit message: changes
Parts:
- removed R6, R7: 49.9, Resistor_SMD:R_0805_2012Metric
- added C8: 0.1uF, Capacitor_SMD:C_0805_2012Metric, B.Cu at (97.0, 93.5)
- added R13: 10k, Resistor_SMD:R_0805_2012Metric, B.Cu at (126.0, 122.9)
- C1: value 1uF -> 0.1uF
- C5: value 1uF -> 2.2uF
- R11, R12: value 4.7k -> 10k
- moved R9 8.16 mm to (117.9, 100.3), turned to 90 degrees
- moved C1 4.65 mm to (109.0, 98.5), turned to 0 degrees
- moved R11 4.15 mm to (145.5, 122.9), turned to 90 degrees
- moved R12 3.28 mm to (145.5, 119.3), turned to -90 degrees
- moved R10 2.97 mm to (117.9, 95.9), turned to 90 degrees
- moved C7 1.20 mm to (154.9, 85.4)
- moved U2 1.20 mm to (113.9, 85.2)
- moved C5 0.17 mm to (139.7, 112.3)
Connections:
- net Net-(IC1-CE) renamed /Batt
- R11 pad 2: /SDA_M -> /SDA
- R12 pad 2: /SCL_M -> /SCL
- U1 pad 8: Net-(U1-SDA) -> /SDA
- U1 pad 9: Net-(U1-SCL) -> /SCL
- U3 pad 7: /SCL_M -> /SCL
- U3 pad 8: /SDA_M -> /SDA
- U4 pad CN3_1: /SCL_M -> /ALERT
- U4 pad CN3_14: /ALERT -> unconnected-(U4-PB5-PadCN3_14)
- U4 pad CN3_2: /SDA_M -> unconnected-(U4-PA10-PadCN3_2)
- U4 pad CN4_5: unconnected-(U4-PA2-PadCN4_5) -> /MISO
- U5 pad 9: unconnected-(U5-MISO-Pad9) -> /MISO
Routing:
- net /SDA: track 60.4 -> 104.3 mm, vias 2 -> 4
- net /SCL: track 57.0 -> 100.2 mm, vias 1 -> 2
- net /ALERT: track 71.8 -> 36.5 mm
- net /MISO: track 0.00 -> 31.6 mm
- net /SCL_M: track 27.8 -> 0.00 mm
- net /SDA_M: track 27.1 -> 0.00 mm
- net /Batt: track 122.6 -> 132.2 mm, vias 7 -> 3
- net GND: track 18.6 -> 13.4 mm, vias 7 -> 8
- net Net-(U1-SCL): track 3.91 -> 0.00 mm
- net Net-(U1-SDA): track 3.90 -> 0.00 mm
- net +3.3V: track 1.22 -> 3.53 mm
- net /V+: track 7.58 -> 9.28 mm
- net Net-(U2-+): track 27.9 -> 29.5 mm
- net /V-: track 1.30 -> 2.86 mm
Other:
- board text added: "+"
- board text added: "-"
